File: PCB/PP.sch (KiCad schematic (older format))
At the start: 10 parts, among them Q1 Q_PMOS_DGS, Q2 Q_NMOS_DGS, Q3 Q_PMOS_DGS, Q4 Q_NMOS_DGS, U1 ESP32-WROOM

Commit message: new pcb! V1
Parts:
- removed D1: LED, LED_THT:LED_D3.0mm_Horizontal_O6.35mm_Z10.0mm, symbol Device:LED
- removed D2: IR, symbol Device:LED
- removed U1: ESP32-WROOM, ESP32-footprints-Lib:ESP32-WROOM, symbol ESP32-footprints-Shem-Lib:ESP32-WROOM
- added 3V3_lux1, 5V_batt1, AT1, AT2, CT1, CT2, GNDT1, GNDT2, GND_BAT1, GNDlux1, MOT1, MOT2, backup_out1, backup_out2, capteurNCbas1, capteurNChaut1, capteur_NC3.3Vbas1, capteur_NC3.3Vhaut1, capteurlux1, remote_AT1, remote_AT2, remote_CT1, remote_CT2, remote_gnd1, remote_gnd2: Conn_01x01, Connector_Pin:Pin_D1.2mm_L11.3mm_W3.0mm_Flat, symbol Connector_Generic:Conn_01x01
- added R4: 10k, Resistor_SMD:R_0603_1608Metric, symbol Device:R
- added R5, R6, R7: 12, Resistor_SMD:R_0603_1608Metric_Pad1.05x0.95mm_HandSolder, symbol Device:R
- added U1: ESP32_DEVKITV1, wemos:devkt1_online, symbol MCU_Espressif:ESP32_DEVKITV1
- added capteurbas1, capteurhaut1: TCRT5000, wemos:TCRT5000, symbol tcrt5000:TCRT5000
- R1: value 21 -> 33; footprint Resistor_SMD:R_0201_0603Metric -> Resistor_SMD:R_0603_1608Metric
- R2: value 34 -> 10k; footprint Resistor_SMD:R_0201_0603Metric -> Resistor_SMD:R_0603_1608Metric
- R3: value MOTEUR -> 33; footprint Resistor_THT:R_Axial_DIN0617_L17.0mm_D6.0mm_P25.40mm_Horizontal -> Resistor_SMD:R_0603_1608Metric
Connections:
- net VCC: now also R2.1, 3V3_lux1.1 (Pin_1), R4.2, U1.30 (VDD), capteur_NC3.3Vbas1.1 (Pin_1), capteur_NC3.3Vhaut1.1 (Pin_1)
- net at Q1.1 (D), Q2.1 (D): now also MOT1.1 (Pin_1); no longer R3.2
- net at Q1.2 (G), Q2.2 (G): now also U1.20 (GPIO021), backup_out1.1 (Pin_1)
- net GND: now reaches Q2.3 (S), Q4.3 (S)
- net GND: now also GNDT1.1 (Pin_1), GNDT2.1 (Pin_1), GND_BAT1.1 (Pin_1), GNDlux1.1 (Pin_1), U1.14 (GND)
- net at Q3.1 (D), Q4.1 (D): now also R5.1, R6.1, R7.1; no longer R3.1
- net at Q3.2 (G), Q4.2 (G): now also U1.25 (GPIO016), backup_out2.1 (Pin_1)
- net 5V: now reaches Q1.3 (S), Q3.3 (S)
- net 5V: now also 5V_batt1.1 (Pin_1), U1.15 (VIN)
- net at R1.2: now also U1.6 (GPIO032)
- net at R2.2: now also CT1.1 (Pin_1)
- net at R1.1: now also AT1.1 (Pin_1)
- new net: U1.2 (ADC1_CH0/VP), capteurlux1.1 (Pin_1)
- new net: U1.4 (GPIO034), capteurNChaut1.1 (Pin_1)
- new net: U1.5 (GPIO035), capteurNCbas1.1 (Pin_1)
- new net: R3.2, U1.7 (GPIO033)
- new net: MOT2.1 (Pin_1), R5.2, R6.2, R7.2
- new net: capteurhaut1.1 (A), remote_AT1.1 (Pin_1)
- new net: capteurhaut1.2 (C), capteurhaut1.4 (E), remote_gnd1.1 (Pin_1)
- new net: capteurhaut1.3 (C), remote_CT1.1 (Pin_1)
- new net: capteurbas1.1 (A), remote_AT2.1 (Pin_1)
- new net: capteurbas1.2 (C), capteurbas1.4 (E), remote_gnd2.1 (Pin_1)
- new net: capteurbas1.3 (C), remote_CT2.1 (Pin_1)
- new net: CT2.1 (Pin_1), R4.1
- new net: AT2.1 (Pin_1), R3.1
Other:
- note added: "For battery"
- note added: "Lux sensor"
